File: LowPass/LowPass.brd (EAGLE design)
At the start: 50.8 x 17.4 mm, 10 parts

Commit message: Update PCB
Routing:
- net N$5: track 28.4 -> 24.2 mm
- net N$3: track 13.9 -> 12.3 mm
- net N$7: track 33.5 -> 32.5 mm
- net N$9: track 6.88 -> 6.13 mm
- removed copper zone on layer 1, net GND

Commit message: Copies PCB
Routing:
- net GND: track 93.7 -> 110.1 mm
Changed lines of the file:
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@@
 <layer number="16" name="Bottom" color="1" fill="1" visible="no" active="yes"/>
 <layer number="17" name="Pads" color="2" fill="1" visible="yes" active="yes"/>
-<layer number="18" name="Vias" color="2" fill="1" visible="no" active="yes"/>
-<layer number="19" name="Unrouted" color="6" fill="1" visible="no" active="yes"/>
+<layer number="18" name="Vias" color="2" fill="1" visible="yes" active="yes"/>
+<layer number="19" name="Unrouted" color="6" fill="1" visible="yes" active="yes"/>
 <layer number="20" name="Dimension" color="24" fill="1" visible="no" active="yes"/>
 <layer number="21" name="tPlace" color="7" fill="1" visible="no" active="yes"/>
@@
 <contactref element="L2" pad="1"/>
 <contactref element="C2" pad="1"/>
-<wire x1="8.89" y1="91.44" x2="13.97" y2="91.44" width="0.8128" layer="1"/>
 <wire x1="13.97" y1="91.44" x2="16.51" y2="93.98" width="0.8128" layer="1"/>
 <wire x1="13.97" y1="91.44" x2="16.51" y2="88.9" width="0.8128" layer="1"/>
+<wire x1="8.89" y1="91.44" x2="13.97" y2="91.44" width="1.27" layer="1"/>
 </signal>
 <signal name="N$5">
@@
 <wire x1="38.1" y1="93.98" x2="40.64" y2="93.98" width="0.8128" layer="1"/>
 <wire x1="40.64" y1="93.98" x2="43.18" y2="91.44" width="0.8128" layer="1"/>
-<wire x1="43.18" y1="91.44" x2="46.99" y2="91.44" width="0.8128" layer="1"/>
 <wire x1="50.8" y1="83.82" x2="48.26" y2="86.36" width="0.8128" layer="1"/>
 <wire x1="48.26" y1="86.36" x2="41.91" y2="86.36" width="0.8128" layer="1"/>
 <wire x1="41.91" y1="86.36" x2="41.91" y2="90.17" width="0.8128" layer="1"/>
 <wire x1="41.91" y1="90.17" x2="43.18" y2="91.44" width="0.8128" layer="1"/>
+<wire x1="46.99" y1="91.44" x2="43.18" y2="91.44" width="1.27" layer="1"/>
 </signal>
 <signal name="N$8">
@@
 <contactref element="SMA2" pad="5"/>
 <contactref element="SMA2" pad="2"/>
-<wire x1="6.4008" y1="93.8784" x2="6.3401" y2="93.9899" width="0.1524" layer="1"/>
 <wire x1="11.43" y1="89.0016" x2="11.4399" y2="88.8901" width="0.1524" layer="16"/>
 <wire x1="6.4008" y1="89.0016" x2="6.346521875" y2="88.90189375" width="0.1524" layer="1"/>
 <wire x1="6.346521875" y1="88.90189375" x2="6.3401" y2="88.8901" width="0.1524" layer="1"/>
-<wire x1="11.43" y1="89.0016" x2="11.43895" y2="88.90079375" width="0.1524" layer="1"/>
-<wire x1="11.43895" y1="88.90079375" x2="11.4399" y2="88.8901" width="0.1524" layer="1"/>
-<wire x1="6.5123" y1="93.9899" x2="6.4008" y2="93.8784" width="0.1524" layer="1"/>
+<wire x1="11.43895" y1="88.90079375" x2="11.43" y2="89.0016" width="0.1524" layer="1"/>
+<wire x1="6.5123" y1="93.9899" x2="6.4262" y2="93.9038" width="0.1524" layer="1"/>
 <contactref element="C4" pad="2"/>
 <contactref element="C5" pad="2"/>
@@
 <contactref element="SMA1" pad="5"/>
 <contactref element="SMA1" pad="2"/>
-<wire x1="49.53" y1="89.0016" x2="49.53895" y2="88.90079375" width="0.1524" layer="1"/>
-<wire x1="49.53895" y1="88.90079375" x2="49.5399" y2="88.8901" width="0.1524" layer="1"/>
 <wire x1="44.4401" y1="88.8901" x2="44.45" y2="88.9" width="0.1524" layer="1"/>
 <wire x1="44.45" y1="88.9" x2="44.45079375" y2="88.90079375" width="0.1524" layer="1"/>
 <wire x1="49.53895" y1="93.98895" x2="49.5399" y2="93.9899" width="0.1524" layer="1"/>
-<wire x1="6.3401" y1="93.9899" x2="11.4399" y2="93.9899" width="0.8128" layer="1"/>
 <wire x1="6.3401" y1="93.9899" x2="6.346521875" y2="93.983478125" width="0.8128" layer="1"/>
-<wire x1="6.346521875" y1="93.983478125" x2="6.346521875" y2="88.90189375" width="0.8128" layer="1"/>
 <wire x1="6.3401" y1="88.8901" x2="6.35079375" y2="88.90079375" width="0.8128" layer="1"/>
-<wire x1="6.35079375" y1="88.90079375" x2="11.43895" y2="88.90079375" width="0.8128" layer="1"/>
 <wire x1="44.4401" y1="93.9899" x2="44.44105" y2="93.98895" width="0.8128" layer="1"/>
 <wire x1="44.44105" y1="93.98895" x2="49.53895" y2="93.98895" width="0.8128" layer="1"/>
-<wire x1="49.5399" y1="88.8901" x2="49.5399" y2="93.988" width="0.8128" layer="1"/>
+<wire x1="49.5399" y1="88.8901" x2="49.5399" y2="93.98" width="0.8128" layer="1"/>
+<wire x1="49.5399" y1="93.98" x2="49.5399" y2="93.988" width="0.8128" layer="1"/>
 <wire x1="49.5399" y1="93.988" x2="49.53895" y2="93.98895" width="0.8128" layer="1"/>
-<wire x1="49.5399" y1="88.8901" x2="49.53" y2="88.9" width="0.8128" layer="1"/>
 <wire x1="49.53" y1="88.9" x2="44.45" y2="88.9" width="0.8128" layer="1"/>
 <wire x1="49.5399" y1="88.8901" x2="53.1676" y2="85.2624" width="0.8128" layer="1"/>
@@
 <wire x1="34.29" y1="82.55" x2="38.1" y2="82.55" width="0.8128" layer="1"/>
 <wire x1="15.24" y1="82.55" x2="34.29" y2="82.55" width="0.8128" layer="1"/>
+<wire x1="11.4399" y1="93.9899" x2="11.3538" y2="93.9038" width="2.54" layer="1"/>
+<wire x1="11.3538" y1="93.9038" x2="6.4262" y2="93.9038" width="2.54" layer="1"/>
+<wire x1="6.3401" y1="93.9899" x2="6.4262" y2="93.9038" width="2.54" layer="1"/>
+<wire x1="6.3401" y1="93.9899" x2="6.35" y2="93.98" width="2.54" layer="1"/>
+<wire x1="6.35" y1="93.98" x2="6.35" y2="92.71" width="2.54" layer="1"/>
+<wire x1="6.35" y1="93.98" x2="6.346521875" y2="93.976521875" width="2.54" layer="1"/>
+<wire x1="6.346521875" y1="93.976521875" x2="6.346521875" y2="88.90189375" width="2.54" layer="1"/>
+<wire x1="11.4399" y1="88.8901" x2="11.43895" y2="88.89105" width="2.54" layer="1"/>
+<wire x1="11.43895" y1="88.89105" x2="11.43895" y2="88.90079375" width="2.54" layer="1"/>
+<wire x1="11.4399" y1="88.8901" x2="11.3284" y2="89.0016" width="2.54" layer="1"/>
+<wire x1="11.3284" y1="89.0016" x2="6.4008" y2="89.0016" width="2.54" layer="1"/>
+<wire x1="44.4401" y1="93.9899" x2="44.45" y2="93.98" width="2.54" layer="1"/>
+<wire x1="44.45" y1="93.98" x2="49.5399" y2="93.98" width="2.54" layer="1"/>
+<wire x1="49.53" y1="93.98" x2="49.5399" y2="93.9899" width="2.54" layer="1"/>
+<wire x1="49.5399" y1="88.8901" x2="49.53" y2="88.9" width="2.54" layer="1"/>
+<wire x1="49.53" y1="88.9" x2="49.53" y2="93.98" width="2.54" layer="1"/>
+<wire x1="44.4401" y1="88.8901" x2="49.5399" y2="88.8901" width="2.54" layer="1"/>
 </signal>
 </signals>

Commit message: Version SMD Reject Band
Parts:
- added C1: 100p, rcl:C0805
- added C10, C9: 10p, rcl:C0805
- added C6: 68p, rcl:C0402
- added C7, C8: 4p, rcl:C1206
- added L1: 12n, inductors:MICC10
- C2: value (none) -> 100p; device rcl:C025-024X044 -> rcl:C0805
- C3: value (none) -> 10p; device rcl:C025-024X044 -> rcl:C0805
- C4: value (none) -> 4p; device rcl:C025-024X044 -> rcl:C1206
- C5: value (none) -> 18p; device rcl:C025-024X044 -> rcl:C0805
- L2: value MICC10 -> 220n
- L3: value MICC10 -> 85n
- L4: value MICC10 -> 500n
- L5: value MICC10 -> 100n
- moved L4 26.2 mm to (49.5, 91.4), turned to 0 degrees
- moved C5 20.7 mm to (24.1, 102.9), turned to 0 degrees
- moved C3 19.8 mm to (17.8, 102.9)
- moved L5 18.8 mm to (28.6, 91.4)
- moved C4 18.5 mm to (43.3, 100.5), flipped to the top, turned to 90 degrees
- moved L2 14.8 mm to (34.3, 101.6), turned to 180 degrees
- moved SMA1 14.0 mm to (61.0, 91.4)
- moved C2 8.89 mm to (17.8, 97.8)
- moved L3 4.49 mm to (38.7, 90.8), turned to 90 degrees
Connections:
- removed net N$7: C3.2, L3.2, L5.2, SMA1.1
- removed net N$9: C5.1, L5.1
- new net N$10: C9.1, L4.1
- new net N$11: C10.1, C9.2
- new net N$12: C4.2, C7.2, C8.2, L2.1
- net GND: now also C10.2, C4.1, C7.1, C8.1; no longer C4.2, C5.2
- net N$3: now also C1.1, C3.1, L1.1; no longer L2.1
- net N$5: now also C1.2, C3.2, C5.1, C6.1, L1.2, L5.1; no longer C3.1, L4.2
- net N$8: now also C5.2, C6.2, L3.2, L4.2, L5.2, SMA1.1; no longer C4.1, L4.1
Routing:
- net N$8: track 2.54 -> 51.3 mm
- net N$5: track 24.2 -> 60.4 mm
- net N$7: track 32.7 -> 0.00 mm
- net N$3: track 12.3 -> 25.9 mm
- net N$12: track 0.00 -> 11.0 mm
- net GND: track 110.1 -> 99.6 mm
- net N$10: track 0.00 -> 6.75 mm
- net N$9: track 6.13 -> 0.00 mm
- net N$11: track 0.00 -> 4.90 mm
Other:
- board size 50.8 x 17.4 mm -> 62.2 x 26.3 mm
- board text added: "Reject Band"
