File: LowPass/LowPass.sch (EAGLE design)
At the start: 10 parts

Commit message: Version SMD Reject Band
Parts:
- added C1: 100p, rcl:C-EUC0805
- added C10, C9: 10p, rcl:C-EUC0805
- added C6: 68p, rcl:C-EUC0402
- added C7, C8: 4p, rcl:C-EUC1206
- added L1: 12n, inductors:MICC10
- C2: value (none) -> 100p; device rcl:C-EU025-024X044 -> rcl:C-EUC0805
- C3: value (none) -> 10p; device rcl:C-EU025-024X044 -> rcl:C-EUC0805
- C4: value (none) -> 4p; device rcl:C-EU025-024X044 -> rcl:C-EUC1206
- C5: value (none) -> 18p; device rcl:C-EU025-024X044 -> rcl:C-EUC0805
- L2: value MICC10 -> 220n
- L3: value MICC10 -> 85n
- L4: value MICC10 -> 500n
- L5: value MICC10 -> 100n
Connections:
- removed net N$7: C3.2, L3.2, L5.2, SMA1.1
- removed net N$9: C5.1, L5.1
- new net N$10: C9.1, L4.1
- new net N$11: C10.1, C9.2
- new net N$12: C4.2, C7.2, C8.2, L2.1
- net GND: now also C10.2, C4.1, C7.1, C8.1; no longer C4.2, C5.2
- net N$3: now also C1.1, C3.1, L1.1; no longer L2.1
- net N$5: now also C1.2, C3.2, C5.1, C6.1, L1.2, L5.1; no longer C3.1, L4.2
- net N$8: now also C5.2, C6.2, L3.2, L4.2, L5.2, SMA1.1; no longer C4.1, L4.1
Other:
- moved on the sheet: C2, C3, C4, C5, L2, L4, L5
